File: pcb/REV10/BusPirate-5-rev10.kicad_pcb (KiCad board)
At the start: 4 copper layers, 60.5 x 60 mm, 220 parts, among them J201 Conn_01x03, J202 TYPE-C-31-M-12, J301 Conn_01x10, J302 Conn_01x09, Q202 2N7002, Q300 SI2301, Q301 SI2301, Q302 SI2301, Q303 SI2301, Q304 SI2301, Q305 SI2301, Q306 SI2301, Q307 SI2301, Q401 BCM857, Q402 SI2301, Q601 MMDT3906, Q602 SI2301, SW101 SW_SPST, SW102 4P_button_sw, U102 W25Q128JVSIQ, U103 RP2040, U105 MT29F1G01ABAFDWB, U301 74LVC1T45, U302 74LVC1T45, U303 74LVC1T45, U304 74LVC1T45, U305 74LVC1T45, U306 74LVC1T45, U307 74LVC1T45, U308 74LVC1T45, U401 ME6211A33PG-N, U402 CD4067, U403 AP2127, U404 LMV321, U501 74HC595, U502 74HC595, U503 74HCT245PW, U504 LMV324, U505 LMV324, U506 LMV321, U601 LMV321A, U602 LMV331, U603 LMV321, Y101 12Mhz

Commit message: making chris branch
Other:
- board text added: "45 degs"
- board text added: "J103"
- board text added: "PIN 1"
